File: KiCAD/ChainSawDIY/ChainSawDIY.sch (KiCad schematic (older format))
At the start: 37 parts, among them J1 BUTTON, J2 BAT_IN, J3 PWR_SW, J4 FAN, J5 MOTOR, J6 PROG, J7 LCD, Q1 PMR280UN, Q2 PMR280UN, Q3 AOD480, U1 ATmega8L-8AU, U2 MAXM15465, U3 MAXM15068

Commit message: Fuse data
Other:
- note added: "Fuses:\nL=A4\nH=D9"
Changed lines of the file:
@@
 Text Notes 3250 3250 0    50   ~ 0
 2.63V
+Text Notes 2200 3800 0    118  ~ 0
+Fuses:\nL=A4\nH=D9
 $EndSCHEMATC
